Commit message: Trying to get the urdf to its final stage....

File: bebop_gazebo/urdf/bebop.urdf.xacro (robot description, xacro)
@@ -13,5 +13,5 @@
   <link name="base_link">
   <inertial>
-    <mass value="0.4" />
+    <mass value="2.477" />
     <origin xyz="0 0 0" />
     <inertia ixx="0.01152" ixy="0.0" ixz="0.0" iyy="0.01152" iyz="0.0" izz="0.0218" />
@@ -65,3 +65,82 @@
       <material>Gazebo/Blue</material>
     </gazebo>
+<gazebo>
+      <plugin name="quadrotor_simple_controller" filename="libhector_gazebo_quadrotor_simple_controller.so">
+        <alwaysOn>true</alwaysOn>
+        <updateRate>10.0</updateRate>
+        <bodyName>base_link</bodyName>
+        <topicName>cmd_vel</topicName>
+        <rollpitchProportionalGain>10.0</rollpitchProportionalGain>
+        <rollpitchDifferentialGain>5.0</rollpitchDifferentialGain>
+        <rollpitchLimit>0.5</rollpitchLimit>
+        <yawProportionalGain>2.0</yawProportionalGain>
+        <yawDifferentialGain>1.0</yawDifferentialGain>
+        <yawLimit>1.5</yawLimit>
+        <velocityXYProportionalGain>5.0</velocityXYProportionalGain>
+        <velocityXYDifferentialGain>1.0</velocityXYDifferentialGain>
+        <velocityXYLimit>2</velocityXYLimit>
+        <velocityZProportionalGain>5.0</velocityZProportionalGain>
+        <velocityZDifferentialGain>1.0</velocityZDifferentialGain>
+        <velocityZLimit>0.5</velocityZLimit>
+        <maxForce>30</maxForce>
+        <motionSmallNoise>0.05</motionSmallNoise>
+        <motionDriftNoise>0.03</motionDriftNoise>
+        <motionDriftNoiseTime>5.0</motionDriftNoiseTime>
+      </plugin>
+      <plugin name="quadrotor_groundtruth_sim" filename="libgazebo_ros_p3d.so">
+        <alwaysOn>true</alwaysOn>
+        <updateRate>100.0</updateRate>
+        <bodyName>base_link</bodyName>
+        <topicName>bebop/odom</topicName>
+        <gaussianNoise>0.0</gaussianNoise>
+        <frameName>/world</frameName>
+      </plugin>
+      <plugin name="quadrotor_aerodynamics" filename="libhector_gazebo_quadrotor_aerodynamics.so">
+        <alwaysOn>true</alwaysOn>
+        <updateRate>100.0</updateRate>
+        <bodyName>base_link</bodyName>
+        <frameId>base_link</frameId>
+      </plugin>
+      <plugin name="quadrotor_propulsion" filename="libhector_gazebo_quadrotor_propulsion.so">
+        <alwaysOn>true</alwaysOn>
+        <updateRate>0.0</updateRate>
+        <bodyName>base_link</bodyName>
+        <frameId>base_link</frameId>
+        <controlRate>100.0</controlRate>
+        <controlTolerance>0.01</controlTolerance>
+        <controlDelay>0.01</controlDelay>
+        <motorStatusRate>0.0</motorStatusRate>
+        <triggerTopic></triggerTopic>
+        <topicName></topicName>
+        <pwmTopicName></pwmTopicName>
+        <supplyTopic></supplyTopic>
+        <wrenchTopic></wrenchTopic>
+        <statusTopic></statusTopic>
+      </plugin>
+    </gazebo>
+<gazebo reference="camera_base_link">
+  <sensor type="camera" name="bebop_camera_sensor">
+        <update_rate>30.0</update_rate>
+        <camera name="front">
+          <horizontal_fov>180</horizontal_fov>
+          <image>
+            <width>640</width>
+            <height>480</height>
+            <format>jpeg</format>
+          </image>
+          <clip>0.01
+            <near>0.01</near>
+            <far>100</far>
+          </clip>
+        </camera>
+        <plugin name="bebop_camera_controller" filename="libgazebo_ros_camera.so">
+    <cameraName>/bebop/camera</cameraName>
+          <alwaysOn>true</alwaysOn>
+          <updateRate>30.0</updateRate>
+          <imageTopicName>/bebop/camera/image_raw</imageTopicName>
+          <cameraInfoTopicName>/bebop/camera/camera_info</cameraInfoTopicName>
+          <frameName>camera_base_link</frameName>
+        </plugin>
+  </sensor>
+    </gazebo>
 </robot>

Commit message: Almost done. Something is wrong with the odom publisher.

File: bebop_gazebo/urdf/bebop.urdf.xacro (robot description, xacro)
@@ -1,146 +1,9 @@
 <?xml version="1.0"?>
-<robot name="bebop" xmlns:xacro="http://www.ros.org/wiki/xacro">
-  <xacro:property name="PI" value="3.1415926535897931" />
-  <xacro:property name="camera_offset_len" value="0.1" />
-  <xacro:property name="camera_offset_ver" value="0.0" />
-  <!-- +- 35 degrees -->
-  <xacro:property name="pan_range" value="0.6108652381980153" />
-  <xacro:property name="pan_vel" value="2.0" />
-  <!-- +- 35 degrees -->
-  <xacro:property name="tilt_range" value="0.6108652381980153" />
-  <xacro:property name="tilt_vel" value="2.0" />
-  <xacro:property name="joint_effort" value="50" />
-  <link name="base_link">
-  <inertial>
-    <mass value="2.477" />
-    <origin xyz="0 0 0" />
-    <inertia ixx="0.01152" ixy="0.0" ixz="0.0" iyy="0.01152" iyz="0.0" izz="0.0218" />
-    <!-- Inertia is just copy-pasted from the hector_quadrotor. Sorry! -->
-  </inertial>
-   <visual>
-      <geometry>
-        <mesh scale="1.0 1.0 1.0" filename="package://bebop_gazebo/meshes/bebop_model.stl"/>
-      </geometry>
-        <material name="blue">
-          <color rgba="0 0.4 0.6 1"/>
-        </material>
-   </visual>
-   <collision>
-      <geometry>
-        <mesh scale="1.0 1.0 1.0" filename="package://bebop_gazebo/meshes/bebop_model.stl"/>
-      </geometry>
-   </collision>
-  </link>
-  <link name="camera_base_link"></link>
-  <link name="camera_pan_link"></link>
-  <link name="camera_tilt_link"></link>
-  <link name="camera_optical"></link>
-  <joint name="base_link_joint" type="fixed">
-    <origin xyz="${camera_offset_len} 0 ${camera_offset_ver}" rpy="0 0 0" />
-    <parent link="base_link"/>
-    <child link="camera_base_link" />
-  </joint>
-  <joint name="camera_pan_joint" type="revolute">
-    <origin xyz="0 0 0" rpy="0 0 0" />
-    <parent link="camera_base_link" />
-    <child link="camera_pan_link" />
-    <axis xyz="0 0 1" />
-    <limit lower="${-pan_range}" upper="${pan_range}"
-      effort="${joint_effort}" velocity="${pan_vel}" />
-  </joint>
-  <joint name="camera_tilt_joint" type="revolute">
-    <origin xyz="0 0 0" rpy="0 0 0" />
-    <parent link="camera_pan_link" />
-    <child link="camera_tilt_link" />
-    <axis xyz="0 1 0" />
-    <limit lower="${-tilt_range}" upper="${tilt_range}"
-      effort="${joint_effort}" velocity="${tilt_vel}" />
-  </joint>
-  <joint name="camera_optical_joint" type="fixed">
-    <origin xyz="0 0 0" rpy="${-PI/2} 0 ${-PI/2}" />
-    <parent link="camera_tilt_link" />
-    <child link="camera_optical" />
-  </joint>
-  <gazebo reference="base_link">
-      <material>Gazebo/Blue</material>
-    </gazebo>
-<gazebo>
-      <plugin name="quadrotor_simple_controller" filename="libhector_gazebo_quadrotor_simple_controller.so">
-        <alwaysOn>true</alwaysOn>
-        <updateRate>10.0</updateRate>
-        <bodyName>base_link</bodyName>
-        <topicName>cmd_vel</topicName>
-        <rollpitchProportionalGain>10.0</rollpitchProportionalGain>
-        <rollpitchDifferentialGain>5.0</rollpitchDifferentialGain>
-        <rollpitchLimit>0.5</rollpitchLimit>
-        <yawProportionalGain>2.0</yawProportionalGain>
-        <yawDifferentialGain>1.0</yawDifferentialGain>
-        <yawLimit>1.5</yawLimit>
-        <velocityXYProportionalGain>5.0</velocityXYProportionalGain>
-        <velocityXYDifferentialGain>1.0</velocityXYDifferentialGain>
-        <velocityXYLimit>2</velocityXYLimit>
-        <velocityZProportionalGain>5.0</velocityZProportionalGain>
-        <velocityZDifferentialGain>1.0</velocityZDifferentialGain>
-        <velocityZLimit>0.5</velocityZLimit>
-        <maxForce>30</maxForce>
-        <motionSmallNoise>0.05</motionSmallNoise>
-        <motionDriftNoise>0.03</motionDriftNoise>
-        <motionDriftNoiseTime>5.0</motionDriftNoiseTime>
-      </plugin>
-      <plugin name="quadrotor_groundtruth_sim" filename="libgazebo_ros_p3d.so">
-        <alwaysOn>true</alwaysOn>
-        <updateRate>100.0</updateRate>
-        <bodyName>base_link</bodyName>
-        <topicName>bebop/odom</topicName>
-        <gaussianNoise>0.0</gaussianNoise>
-        <frameName>/world</frameName>
-      </plugin>
-      <plugin name="quadrotor_aerodynamics" filename="libhector_gazebo_quadrotor_aerodynamics.so">
-        <alwaysOn>true</alwaysOn>
-        <updateRate>100.0</updateRate>
-        <bodyName>base_link</bodyName>
-        <frameId>base_link</frameId>
-      </plugin>
-      <plugin name="quadrotor_propulsion" filename="libhector_gazebo_quadrotor_propulsion.so">
-        <alwaysOn>true</alwaysOn>
-        <updateRate>0.0</updateRate>
-        <bodyName>base_link</bodyName>
-        <frameId>base_link</frameId>
-        <controlRate>100.0</controlRate>
-        <controlTolerance>0.01</controlTolerance>
-        <controlDelay>0.01</controlDelay>
-        <motorStatusRate>0.0</motorStatusRate>
-        <triggerTopic></triggerTopic>
-        <topicName></topicName>
-        <pwmTopicName></pwmTopicName>
-        <supplyTopic></supplyTopic>
-        <wrenchTopic></wrenchTopic>
-        <statusTopic></statusTopic>
-      </plugin>
-    </gazebo>
-<gazebo reference="camera_base_link">
-  <sensor type="camera" name="bebop_camera_sensor">
-        <update_rate>30.0</update_rate>
-        <camera name="front">
-          <horizontal_fov>180</horizontal_fov>
-          <image>
-            <width>640</width>
-            <height>480</height>
-            <format>jpeg</format>
-          </image>
-          <clip>0.01
-            <near>0.01</near>
-            <far>100</far>
-          </clip>
-        </camera>
-        <plugin name="bebop_camera_controller" filename="libgazebo_ros_camera.so">
-    <cameraName>/bebop/camera</cameraName>
-          <alwaysOn>true</alwaysOn>
-          <updateRate>30.0</updateRate>
-          <imageTopicName>/bebop/camera/image_raw</imageTopicName>
-          <cameraInfoTopicName>/bebop/camera/camera_info</cameraInfoTopicName>
-          <frameName>camera_base_link</frameName>
-        </plugin>
-  </sensor>
-    </gazebo>
+<robot
+  name="quadrotor"
+  xmlns:xacro="http://www.ros.org/wiki/xacro"
+>
+    <!-- Included URDF Files -->
+    <xacro:include filename="$(find bebop_gazebo)/urdf/bebop_base.urdf.xacro" />
+    <xacro:bebop_base_macro />
 </robot>
